File: interleaved-400W-buck.kicad_sch (KiCad schematic)
At the start: 0 parts

Commit message: schematic init
Parts:
- added U1: STM32G474CBTx, Package_QFP:LQFP-48_7x7mm_P0.5mm, symbol MCU_ST_STM32G4:STM32G474CBTx
- added U2: TCAN330, Package_SO:SOIC-8_3.9x4.9mm_P1.27mm, symbol Interface_CAN_LIN:TCAN330
Connections:
- new net: U1.23 (VSS), U1.35 (VSS), U1.47 (VSS)

Commit message: schematic
Parts:
- added U3: LTC7891RUFDM, jannett_footprints:QFN50P500X400X80-29N, symbol jannett_symbols:LTC7891RUFDM
Connections:
- net GND: now reaches U2.2 (GND)
- net GND: now also U1.19 (VSSA), U1.23 (VSS), U1.35 (VSS), U1.47 (VSS), U3.29 (GND)
Other:
- moved on the sheet: U2
